Commit message: Update rg2 gripper urdf xacro

File: rg2_gripper_description/urdf/rg2_gripper.urdf.xacro (robot description, xacro)
@@ -137,5 +137,5 @@
                 </geometry>
             </collision>
-            <contact_coefficients kd="1.0" kp="1000.0" mu="0"/>
+            <contact_coefficients kd="1.0" kp="1000.0" mu="1000"  mu2="1000"/>
         </link>
         <!-- FINGER RIGHT -->
@@ -147,4 +147,5 @@
             <child link="${prefix}_right_finger" />
             <dynamics damping="0" friction="0"/>
+            <mimic joint="${prefix}_finger_left_joint" multiplier="-1.0" offset="0"/>
         </joint>
         <xacro:mimic_joint_plugin_gazebo parent_joint="${prefix}_finger_left_joint"
@@ -214,51 +215,6 @@
                 </geometry>
             </collision>
-            <contact_coefficients kd="1.0" kp="1000.0" mu="0"/>
-        </link>
-        <!--
-        <joint name="${prefix}_finger_right_joint" type="prismatic">
-            <limit lower="0.0" upper="0.048" effort="1.0" velocity="0.0125"/>
-            <axis xyz="0 1 0"/>
-            <origin xyz="0.11 0.013 0" rpy="0 0 0" />
-            <parent link="${prefix}_base_link"/>
-            <child link="${prefix}_right_finger" />
-            <dynamics friction="100" damping="100" />
-            <mimic joint="${prefix}_finger_left_joint" multiplier="1" offset="0"/>
-        </joint>
-        -->
-<!--
-        <xacro:mimic_joint_plugin_gazebo parent_joint="${prefix}_finger_left_joint"
-        mimic_joint="${prefix}_finger_right_joint" has_pid="false" multiplier="1.0"
-        max_effort="10.0" />
-        <link name="${prefix}_right_finger">
-            <inertial>
-            <mass value="0.1" />
-                <origin xyz="0 0 0" />
-                <inertia ixx="1.0" ixy="0.0" ixz="0.0"
-                        iyy="1.0" iyz="0.0"
-                        izz="1.0" />
-            </inertial>
-            <visual>
-                <origin xyz="0.0 0 0" rpy="0 0 0" />
-                <geometry>
-                    <mesh filename="package://rg2_gripper_description/meshes/rg2_finger.stl" scale="1.0 1.0 1.0"/>
-                </geometry>
-                <material name="black">
-                <color rgba="0.2 0.2 0.2 1.0"/>
-                </material>
-            </visual>
-            <collision>
-                <origin xyz="0 0 0" rpy="0 0 0" />
-                <geometry>
-                    <mesh filename="package://rg2_gripper_description/meshes/rg2_finger.stl" scale="1.0 1.0 1.0"/>
-                </geometry>
-            </collision>
-            <contact_coefficients kd="1.0" kp="1000.0" mu="0"/>
-        </link>
-        <gazebo reference="${prefix}_right_finger">
-            <material>Gazebo/Blue</material>
-            <turnGravityOff>false</turnGravityOff>
-        </gazebo>
--->
+            <contact_coefficients kd="1.0" kp="1000.0" mu="1000" mu2="1000"/>
+        </link>
     </xacro:macro>
 </robot>
